File: lower/lower.kicad_pcb (KiCad board)
At the start: 2 copper layers, 177.8 x 127 mm, 4 parts

Commit message: Lower v0.1.0. Pre-routing
Parts:
- added B1: board-outline, lower-all:board-outline-test, F.Cu at (74.0, 153.0)
- added D1: 2.7V, Diode_THT:D_T-1_P5.08mm_Horizontal, B.Cu at (174.1, 63.0)
- added D2: 1N4007, Diode_THT:D_DO-41_SOD81_P10.16mm_Horizontal, B.Cu at (174.2, 57.0)
- added ESCWires1: ~, lower-all:WireESC, F.Cu at (236.0, 40.5)
- added ESCWires2: ~, lower-all:WireESC, F.Cu at (239.0, 135.5)
- added ESCWires3: ~, lower-all:WireESC, F.Cu at (94.0, 134.5)
- added ESCWires4: ~, lower-all:WireESC, F.Cu at (96.0, 40.5)
- added M1: MotorCutout, lower-all:MotorEdges, F.Cu at (250.5, 34.0)
- added M2: MotorCutout, lower-all:MotorEdges, F.Cu at (250.5, 142.9)
- added M3: MotorCutout, lower-all:MotorEdges, F.Cu at (83.5, 142.9)
- added M4: MotorCutout, lower-all:MotorEdges, F.Cu at (84.4, 34.5)
- added MotorWires1: ~, lower-all:WireMotor, F.Cu at (223.0, 28.5)
- added MotorWires2: ~, lower-all:WireMotor, F.Cu at (222.0, 146.5)
- added MotorWires3: ~, lower-all:WireMotor, F.Cu at (113.0, 145.5)
- added MotorWires4: ~, lower-all:WireMotor, F.Cu at (107.0, 28.5)
- added R1: 510, Resistor_SMD:R_0201_0603Metric_Pad0.64x0.40mm_HandSolder, B.Cu at (178.3, 57.0)
- added R2: 33, Resistor_THT:R_Axial_DIN0207_L6.3mm_D2.5mm_P7.62mm_Horizontal, B.Cu at (179.0, 68.6)
- added R3: 470, Resistor_THT:R_Axial_DIN0207_L6.3mm_D2.5mm_P7.62mm_Horizontal, B.Cu at (183.0, 61.0)
- added SW1: SW_SPDT, Button_Switch_THT:SW_Slide_SPDT_Angled_CK_OS102011MA1Q, F.Cu at (189.0, 91.9)
- added TP1: Psense, TestPoint:TestPoint_2Pads_Pitch2.54mm_Drill0.8mm, F.Cu at (190.0, 49.5)
- added U1: BTS50080-1TMA, Package_TO_SOT_SMD:TO-263-7_TabPin4, B.Cu at (166.8, 42.9)
- added WireBatt1: ~, lower-all:WireBatt, F.Cu at (167.0, 29.0)
- added WireESCPwr1: ~, lower-all:WireESCPwr, F.Cu at (178.0, 50.0)
- added WireESCPwr2: ~, lower-all:WireESCPwr, F.Cu at (178.0, 129.5)
- added WireESCPwr3: ~, lower-all:WireESCPwr, F.Cu at (154.0, 129.5)
- added WireESCPwr4: ~, lower-all:WireESCPwr, F.Cu at (154.0, 50.0)
- H1, H2, H3, H4: value MountingHole_Pad -> MountingHole
- moved H4 127.0 mm to (152.0, 28.0)
- moved H2 114.4 mm to (181.0, 149.0)
- moved H1 62.1 mm to (181.0, 28.0)
- moved H3 32.7 mm to (152.0, 149.0)
Routing:
- net /C1: track 0.00 -> 18.0 mm
- net /B1: track 0.00 -> 18.0 mm
- net /A1: track 0.00 -> 18.0 mm
- net /Vbb: track 0.00 -> 2.83 mm
Other:
- board size 177.8 x 127 mm -> 187 x 130 mm
- board text added: "!NOTHING SHOULD POKE BATTERY!"
- board text added: "Battery"
- board text added: "ESC1"
- board text added: "ESC2"
- board text added: "ESC3"
- board text added: "ESC4"
- board text added: "FRONT"
- board text added: "I"
- board text added: "M1"
- board text added: "M2"
- board text added: "M3"
- board text added: "M4"
- board text added: "O"

Commit message: Lower v0.1.1. Pre-routing
Parts:
- added JP1: Jumper_2_Bridged, lower-all:SolderJumperLarge, F.Cu at (153.0, 40.8)
- moved D1 3.08 mm to (171.0, 63.0)
- moved R2 1.00 mm to (178.0, 68.6)
- moved R3 1.00 mm to (182.0, 61.0)
Connections:
- WireBatt1 pad 2: GND -> GNDPWR
- WireESCPwr1 pad 2: GND -> GNDPWR
- WireESCPwr2 pad 2: GND -> GNDPWR
- WireESCPwr3 pad 2: GND -> GNDPWR
- WireESCPwr4 pad 2: GND -> GNDPWR
Routing:
- net /C1: track 18.0 -> 0.00 mm
- net /B1: track 18.0 -> 0.00 mm
- net /A1: track 18.0 -> 0.00 mm
- net /Vbb: track 2.83 -> 0.00 mm

Commit message: Lower v0.1.2. Pre-routing
Parts:
- removed WireBatt1: ~, lower-all:WireBatt
- added Batt1: ~, lower-all:WireBatt, F.Cu at (166.5, 28.0)
- moved MotorWires3 4.61 mm to (108.5, 146.5)
- moved R2 2.00 mm to (176.0, 68.6)
- moved MotorWires4 1.50 mm to (108.5, 28.5)
- moved M2 1.46 mm to (251.0, 141.5)
- moved M3 1.44 mm to (83.0, 141.5)
- moved M4 1.38 mm to (83.0, 34.5)
- moved U1 1.08 mm to (166.8, 44.0)
- moved D1 1.00 mm to (171.0, 64.0)
- moved D2 1.00 mm to (174.2, 58.0)
- moved MotorWires1 1.00 mm to (222.0, 28.5)
- moved M1 0.71 mm to (251.0, 34.5)
- moved WireESCPwr3 0.50 mm to (154.5, 129.5)
- moved WireESCPwr4 0.50 mm to (154.5, 50.0)
Other:
- outline, holes or cut-outs redrawn
- board text removed: "M1"

Commit message: v0.1.2. Routed
Parts:
- moved H1 3.00 mm to (184.0, 28.0)
- moved H2 3.00 mm to (184.0, 149.0)
- moved H3 2.00 mm to (150.0, 149.0)
- moved H4 2.00 mm to (150.0, 28.0)
Routing:
- net GNDPWR: track 0.00 -> 198.7 mm, vias 0 -> 1
- net /Vcc: track 0.00 -> 151.3 mm
- net GND: track 0.00 -> 127.5 mm
- net Net-(SW1-B): track 0.00 -> 47.8 mm
- net /Vbb: track 0.00 -> 37.5 mm
- net /Psense: track 0.00 -> 33.6 mm
- net /C2: track 0.00 -> 21.6 mm
- net /B2: track 0.00 -> 21.6 mm
- net /A2: track 0.00 -> 21.6 mm
- net /C3: track 0.00 -> 19.5 mm
- net /B3: track 0.00 -> 19.5 mm
- net /A3: track 0.00 -> 19.5 mm
- net /C1: track 0.00 -> 19.0 mm
- net /B1: track 0.00 -> 19.0 mm
- net /A1: track 0.00 -> 19.0 mm
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Other:
- outline, holes or cut-outs redrawn
- board text added: "G"
- board text added: "P"

Commit message: Upper/Lower: v0.2.0. Pre-routed
Parts:
- added R4: 0, Resistor_SMD:R_1206_3216Metric_Pad1.30x1.75mm_HandSolder, B.Cu at (192.0, 39.5)
- added R5: 0, Resistor_SMD:R_1206_3216Metric_Pad1.30x1.75mm_HandSolder, B.Cu at (192.1, 43.5)
- added R6: 0, Resistor_THT:R_Axial_DIN0207_L6.3mm_D2.5mm_P7.62mm_Horizontal, B.Cu at (197.6, 30.0)
- added R7: 0, Resistor_THT:R_Axial_DIN0207_L6.3mm_D2.5mm_P7.62mm_Horizontal, B.Cu at (190.0, 34.8)
- added TP2: Vsense, TestPoint:TestPoint_2Pads_Pitch2.54mm_Drill0.8mm, F.Cu at (190.2, 49.5)
- TP1: value Psense -> Isense
- moved TP1 2.50 mm to (187.5, 49.5)
Connections:
- net /Psense renamed /Isense
Routing:
- net GNDPWR: track 198.7 -> 0.00 mm, vias 1 -> 0
- net /Vcc: track 151.3 -> 0.00 mm
- net GND: track 127.5 -> 0.00 mm
- net Net-(SW1-B): track 47.8 -> 0.00 mm
- net /Vbb: track 37.5 -> 0.00 mm
- net /Isense: track 33.6 -> 0.00 mm
- net /C2: track 21.6 -> 0.00 mm
- net /B2: track 21.6 -> 0.00 mm
- net /A2: track 21.6 -> 0.00 mm
- net /C3: track 19.5 -> 0.00 mm
- net /B3: track 19.5 -> 0.00 mm
- net /A3: track 19.5 -> 0.00 mm
- net /C1: track 19.0 -> 0.00 mm
- net /B1: track 19.0 -> 0.00 mm
- net /A1: track 19.0 -> 0.00 mm
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Other:
- board text added: "Isense"
- board text added: "S"
- board text added: "Vsense"
- board text removed: "P"

Commit message: Upper/Lower: v0.2.0. Routed
Routing:
- net /Vcc: track 0.00 -> 179.7 mm
- net GNDPWR: track 0.00 -> 169.9 mm
- net GND: track 0.00 -> 117.0 mm
- net Net-(SW1-B): track 0.00 -> 70.3 mm
- net /Vbb: track 0.00 -> 35.4 mm
- net /Isense: track 0.00 -> 31.7 mm
- net /C2: track 0.00 -> 21.6 mm
- net /A2: track 0.00 -> 21.6 mm
- net /B2: track 0.00 -> 21.6 mm
- net /_Vsense: track 0.00 -> 19.8 mm
- net /C3: track 0.00 -> 19.5 mm
- net /A3: track 0.00 -> 19.5 mm
- net /B3: track 0.00 -> 19.5 mm
- net /C1: track 0.00 -> 19.0 mm
- net /B1: track 0.00 -> 19.0 mm
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
Commit message: Lower: v0.2.1. Routed
Routing:
- net /Vbb: track 35.4 -> 24.1 mm
Changed lines of the file:
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@@
 			(drillshape 0)
 			(scaleselection 1)
-			(outputdirectory "C:/Users/engi/Documents/kicad_projects/nano_quadcopter/lower/lower_v0.1.0/")
+			(outputdirectory "C:/Users/engi/Documents/kicad_projects/nano_quadcopter/lower/v0.2.0/")
 		)
 	)
@@
 	)
 	(segment
-		(start 167.125 42.5)
-		(end 169.55 44.925)
-		(width 3)
-		(layer "B.Cu")
-		(net 7)
-	)
-	(segment
-		(start 164.0264 44.8986)
-		(end 166.775 47.6473)
-		(width 3)
-		(layer "B.Cu")
-		(net 7)
-	)
-	(segment
 		(start 164 40.075)
 		(end 166.425 42.5)
@@
 		(layer "B.Cu")
 		(net 7)
-	)
-	(segment
-		(start 166.775 47.6473)
-		(end 166.775 51.65)
-		(width 0.8014)
-		(layer "B.Cu")
-		(net 7)
