File: lower/lower.kicad_sch (KiCad schematic)
At the start: 36 parts, among them M1 MotorCutout, M2 MotorCutout, M3 MotorCutout, M4 MotorCutout, SW1 SW_SPDT, U1 BTS50080-1TMA

Commit message: Lower: Identify CW/CCW propellor in schematics
From the top down:
* CCW is 3025
* CW is 3025R
Other:
- note added: "3025 Propellor"
- note added: "3025R Propellor"
Changed lines of the file:
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@@
+		)
+	)
+	(text "3025 Propellor"
+		(exclude_from_sim no)
+		(at 127 33.02 0)
+		(effects
+			(font
+				(size 1.27 1.27)
+			)
+		)
+	)
+	(text "3025 Propellor"
+		(exclude_from_sim no)
+		(at 86.106 72.136 0)
+		(effects
+			(font
+				(size 1.27 1.27)
+			)
 		)
 	)
@@
 		)
 	)
+	(text "3025R Propellor"
+		(exclude_from_sim no)
+		(at 86.36 33.528 0)
+		(effects
+			(font
+				(size 1.27 1.27)
+			)
+		)
+	)
+	(text "3025R Propellor"
+		(exclude_from_sim no)
+		(at 128.27 72.136 0)
+		(effects
+			(font
+				(size 1.27 1.27)
+			)
+		)
+	)
